Commit message: ✨ feat: adjusted scenes

File: entities/robots/jackal/urdf/jackal.urdf.xacro (robot description, xacro)
@@ -232,5 +232,5 @@
   <xacro:sensor_d415 name="d415" parent="base_link" use_nominal_extrinsics="true">
     <!-- <origin xyz="0.061 0.0 0.271" rpy="0 0 0"/> -->
-    <origin xyz="0.061 0.0 1.500" rpy="0 0 0"/>
+    <origin xyz="0.061 0.0 0.500" rpy="0 0 0"/>
   </xacro:sensor_d415>
 </robot>

Commit message: ✨ feat: task2-5

File: entities/robots/jackal/urdf/jackal.urdf.xacro (robot description, xacro)
@@ -232,5 +232,5 @@
   <xacro:sensor_d415 name="d415" parent="base_link" use_nominal_extrinsics="true">
     <!-- <origin xyz="0.061 0.0 0.271" rpy="0 0 0"/> -->
-    <origin xyz="0.061 0.0 0.500" rpy="0 0 0"/>
+    <origin xyz="0.061 0.0 1.500" rpy="0 0 0"/>
   </xacro:sensor_d415>
 </robot>

Commit message: ✨ feat: 0911 dev

File: entities/robots/jackal/urdf/jackal.urdf.xacro (robot description, xacro)
@@ -232,5 +232,5 @@
   <xacro:sensor_d415 name="d415" parent="base_link" use_nominal_extrinsics="true">
     <!-- <origin xyz="0.061 0.0 0.271" rpy="0 0 0"/> -->
-    <origin xyz="0.061 0.0 1.500" rpy="0 0 0"/>
+    <origin xyz="0.061 0.0 1.500" rpy="0 0.2 0"/>
   </xacro:sensor_d415>
 </robot>
